File: Kicad Source Files/eavesdrop Receiver/eavesdrop2.kicad_pcb (KiCad board)
At the start: 2 copper layers, 70 x 50 mm, 25 parts, among them J1 Conn_01x02_Pin, M2 MountingHole_2.2mm_M2, T1 ED8_4, U3 LM386

Commit message: fixed an issue with GND of  the receiver circuit
Routing:
- net GND: track 0.00 -> 61.2 mm, vias 0 -> 11
